File: Solar Board.kicad_sch (KiCad schematic)
At the start: 15 parts

Commit message: Update Solar Board.kicad_sch
Parts:
- removed C8: 100nF, Capacitor_SMD:C_0805_2012Metric, symbol Device:C
- removed R10, R11, R12: 10k, Resistor_SMD:R_0603_1608Metric, symbol Device:R_US
- added C1: 100nF, Capacitor_SMD:C_0805_2012Metric, symbol Device:C
- added R4: 0.01, symbol Device:R_US
- added R5, R6: 10k, symbol Device:R_US
- added TP1: Sensor Input, symbol Connector:TestPoint
- added TP2: Rail Voltage, symbol Connector:TestPoint
- added TP3: Shunt Voltage, symbol Connector:TestPoint
- added TP4: SDA, symbol Connector:TestPoint
- added TP5: SCL, symbol Connector:TestPoint
- added TP6, TP7: Alert, symbol Connector:TestPoint
- R1: value 0.01 -> 10k
- R3: value 1k -> 10k
- R7, R8: footprint Resistor_SMD:R_0603_1608Metric -> (none)
- R9: value 10k -> 1k; footprint Resistor_SMD:R_0603_1608Metric -> (none)
- renumbered C7 to C2, C9 to C3, Voltage_Current_Sensor to U1, Temp_Sensor1 to U2, Light_Sensor to U3
Connections:
- net +3.3V: now also R1.2, R2.1, R3.2, R8.2, C1.2, R5.1, R5.2, R6.1, R6.2, TP2.1, TP4.1, TP5.1; no longer R2.2, R8.1, R9.1, R9.2
- net +VIN: now also R4.1, TP1.1; no longer R1.2
- net GND: now also C1.1
- net at C2.1, C3.1, U2.5 (ALERT): now also R7.2, R9.2, TP7.1; no longer R3.1
- net at U2.1 (AS): now also R9.1; no longer R3.2
- net at U1.4 (SDA): now also R2.2
- net at U1.13 (IN+): now also R4.2, TP3.1; no longer R1.1
- net at U1.3 (ALERT): now also R1.1, TP6.1; no longer R7.2
- net at U1.5 (SCL): now also R3.1; no longer R8.2
- net at U3.5 (INT): now also R8.1; no longer R2.1
Other:
- note added: "Light Sensor"
- note added: "Temperature Sensor"
- note added: "Voltage/Current Sensor"
